Commit message: Changed robot definition to reflect reality

File: description/gazebo_control.xacro (robot description, xacro)
@@ -6,9 +6,9 @@
       <left_joint>left_wheel_joint</left_joint>
       <right_joint>right_wheel_joint</right_joint>
-      <wheel_separation>0.13</wheel_separation>
-      <wheel_diameter>0.05</wheel_diameter>
+      <wheel_separation>0.146</wheel_separation>
+      <wheel_diameter>0.08</wheel_diameter>
       <!-- Limits -->
       <max_wheel_torque>2</max_wheel_torque>
-      <max_wheel_acceleration>1.0</max_wheel_acceleration>
+      <max_wheel_acceleration>1</max_wheel_acceleration>
       <!-- Output -->
       <odometry_frame>odom</odometry_frame>

File: description/robot_core.xacro (robot description, xacro)
@@ -18,8 +18,8 @@
   </link>
   <!-- CHASSIS LINK -->
-  <joint name="chassis_join" type="fixed">
+  <joint name="chassis_joint" type="fixed">
     <parent link="base_link" />
     <child link="chassis" />
-    <origin xyz="-0.05 0 0" />
+    <origin xyz="-0.025 0 0.025" />
   </joint>
   <link name="chassis">
@@ -48,5 +48,5 @@
     <parent link="base_link" />
     <child link="left_wheel" />
-    <origin xyz="0 0.065 0" rpy="-${pi/2} 0 0" />
+    <origin xyz="0 0.072 0" rpy="-${pi/2} 0 0" />
     <axis xyz="0 0 1" />
   </joint>
@@ -54,5 +54,5 @@
     <visual>
       <geometry>
-        <cylinder radius="0.025" length="0.02" />
+        <cylinder radius="0.04" length="0.009" />
       </geometry>
       <material name="blue" />
@@ -60,8 +60,8 @@
     <collision>
       <geometry>
-        <cylinder radius="0.025" length="0.02" />
+        <cylinder radius="0.04" length="0.009" />
       </geometry>
     </collision>
-    <xacro:inertial_cylinder mass="0.1" length="0.02" radius="0.025">
+    <xacro:inertial_cylinder mass="0.1" length="0.009" radius="0.04">
       <origin xyz="0 0 0" rpy="0 0 0"/>
     </xacro:inertial_cylinder>
@@ -74,5 +74,5 @@
     <parent link="base_link" />
     <child link="right_wheel" />
-    <origin xyz="0 -0.065 0" rpy="${pi/2} 0 0" />
+    <origin xyz="0 -0.072 0" rpy="${pi/2} 0 0" />
     <axis xyz="0 0 -1" />
   </joint>
@@ -80,5 +80,5 @@
     <visual>
       <geometry>
-        <cylinder radius="0.025" length="0.02" />
+        <cylinder radius="0.04" length="0.009" />
       </geometry>
       <material name="blue" />
@@ -86,8 +86,8 @@
     <collision>
       <geometry>
-        <cylinder radius="0.025" length="0.02" />
+        <cylinder radius="0.04" length="0.009" />
       </geometry>
     </collision>
-    <xacro:inertial_cylinder mass="0.1" length="0.02" radius="0.025">
+    <xacro:inertial_cylinder mass="0.1" length="0.009" radius="0.04">
       <origin xyz="0 0 0" rpy="0 0 0"/>
     </xacro:inertial_cylinder>
@@ -100,10 +100,10 @@
     <parent link="chassis" />
     <child link="caster_wheel" />
-    <origin xyz="0.15 0 0" />
+    <origin xyz="0.15 0 -0.025" />
   </joint>
   <link name="caster_wheel">
     <visual>
       <geometry>
-        <sphere radius="0.025" />
+        <sphere radius="0.04" />
       </geometry>
       <material name="black" />
@@ -111,8 +111,8 @@
     <collision>
       <geometry>
-        <sphere radius="0.025" />
+        <sphere radius="0.04" />
       </geometry>
     </collision>
-    <xacro:inertial_sphere mass="0.1" radius="0.025">
+    <xacro:inertial_sphere mass="0.1" radius="0.04">
       <origin xyz="0 0 0" rpy="0 0 0"/>
     </xacro:inertial_sphere>
