Commit message: Added lidar URDF definitions

File: description/robot.urdf.xacro (robot description, xacro)
@@ -3,3 +3,4 @@
     <xacro:include filename="robot_core.xacro" />
     <xacro:include filename="gazebo_control.xacro"/>
+    <xacro:include filename="lidar.xacro"/>
 </robot>

File: description/robot_core.xacro (robot description, xacro)
@@ -13,4 +13,7 @@
   <material name="black">
     <color rgba="0 0 0 1" />
+  </material>
+  <material name="red">
+    <color rgba="1 0 0 1" />
   </material>
   <!-- BASE LINK -->

Commit message: Added some support for slam_toolbox

File: description/robot.urdf.xacro (robot description, xacro)
@@ -2,4 +2,5 @@
 <robot xmlns:xacro="http://www.ros.org/wiki/xacro"  name="robot">
     <xacro:arg name="use_ros2_control" default="true"/>
+    <xacro:arg name="sim_mode" default="false"/>
     <xacro:include filename="robot_core.xacro" />
     <xacro:if value="$(arg use_ros2_control)">

File: description/robot_core.xacro (robot description, xacro)
@@ -19,4 +19,11 @@
   <!-- BASE LINK -->
   <link name="base_link">
+  </link>
+  <joint name="base_footprint_joint" type="fixed">
+    <parent link="base_link"/>
+    <child link="base_footprint"/>
+    <origin xyz="0 0 0" rpy="0 0 0"/>
+  </joint>
+  <link name="base_footprint">
   </link>
   <!-- CHASSIS LINK -->

File: description/ros2_control.xacro (robot description, xacro)
@@ -1,57 +1,62 @@
 <?xml version="1.0"?>
 <robot xmlns:xacro="http://www.ros.org/wiki/xacro">
-  <ros2_control name="RealRobot" type="system">
-    <hardware>
-      <plugin>diffdrive_arduino/DiffDriveArduino</plugin>
-      <param name="left_wheel_name">left_wheel_joint</param>
-      <param name="right_wheel_name">right_wheel_joint</param>
-      <param name="loop_rate">30</param>
-      <param name="device">/dev/serial/by-id/usb-Espressif_Systems_UNO_WiFi_R4_CMSIS-DAP_DC5475C68794-if01</param>
-      <param name="baud_rate">1000000</param>
-      <param name="timeout">1000</param>
-      <param name="enc_counts_per_rev">3200</param>
-    </hardware>
-    <joint name="left_wheel_joint">
-      <command_interface name="velocity">
-        <param name="min">-10</param>
-        <param name="max">10</param>
-      </command_interface>
-      <state_interface name="velocity"/>
-      <state_interface name="position"/>
-    </joint>
-    <joint name="right_wheel_joint">
-      <command_interface name="velocity">
-        <param name="min">-10</param>
-        <param name="max">10</param>
-      </command_interface>
-      <state_interface name="velocity"/>
-      <state_interface name="position"/>
-    </joint>
-  </ros2_control>
-  <!-- <ros2_control name="GazeboSystem" type="system">
-    <hardware>
-      <plugin>gazebo_ros2_control/GazeboSystem</plugin>
-    </hardware>
-    <joint name="left_wheel_joint">
-      <command_interface name="velocity">
-        <param name="min">-10</param>
-        <param name="max">10</param>
-      </command_interface>
-      <state_interface name="velocity"/>
-      <state_interface name="position"/>
-    </joint>
-    <joint name="right_wheel_joint">
-      <command_interface name="velocity">
-        <param name="min">-10</param>
-        <param name="max">10</param>
-      </command_interface>
-      <state_interface name="velocity"/>
-      <state_interface name="position"/>
-    </joint>
-  </ros2_control> -->
-  <gazebo>
-    <plugin name="gazebo_ros2_control" filename="libgazebo_ros2_control.so">
-      <parameters>$(find slambot)/config/my_controllers.yaml</parameters>
-    </plugin>
-  </gazebo>
+  <xacro:unless value="$(arg sim_mode)">
+    <ros2_control name="RealRobot" type="system">
+      <hardware>
+        <plugin>diffdrive_arduino/DiffDriveArduino</plugin>
+        <param name="left_wheel_name">left_wheel_joint</param>
+        <param name="right_wheel_name">right_wheel_joint</param>
+        <param name="loop_rate">30</param>
+        <param name="device">/dev/serial/by-id/usb-Espressif_Systems_UNO_WiFi_R4_CMSIS-DAP_DC5475C68794-if01</param>
+        <param name="baud_rate">1000000</param>
+        <param name="timeout">1000</param>
+        <param name="enc_counts_per_rev">3200</param>
+      </hardware>
+      <joint name="left_wheel_joint">
+        <command_interface name="velocity">
+          <param name="min">-10</param>
+          <param name="max">10</param>
+        </command_interface>
+        <state_interface name="velocity"/>
+        <state_interface name="position"/>
+      </joint>
+      <joint name="right_wheel_joint">
+        <command_interface name="velocity">
+          <param name="min">-10</param>
+          <param name="max">10</param>
+        </command_interface>
+        <state_interface name="velocity"/>
+        <state_interface name="position"/>
+      </joint>
+    </ros2_control>
+  </xacro:unless>
+  <xacro:if value="$(arg sim_mode)">
+    <ros2_control name="GazeboSystem" type="system">
+      <hardware>
+        <plugin>gazebo_ros2_control/GazeboSystem</plugin>
+      </hardware>
+      <joint name="left_wheel_joint">
+        <command_interface name="velocity">
+          <param name="min">-10</param>
+          <param name="max">10</param>
+        </command_interface>
+        <state_interface name="velocity"/>
+        <state_interface name="position"/>
+      </joint>
+      <joint name="right_wheel_joint">
+        <command_interface name="velocity">
+          <param name="min">-10</param>
+          <param name="max">10</param>
+        </command_interface>
+        <state_interface name="velocity"/>
+        <state_interface name="position"/>
+      </joint>
+    </ros2_control>
+    <gazebo>
+      <plugin name="gazebo_ros2_control" filename="libgazebo_ros2_control.so">
+        <parameters>$(find slambot)/config/my_controllers.yaml</parameters>
+        <parameters>$(find slambot)/config/gaz_ros2_control_use_sim.yaml</parameters>
+      </plugin>
+    </gazebo>
+  </xacro:if>
 </robot>
