Commit message: Added toggle between ros2_control and gazebo_control in sim launch. Also some xacro-fixes

File: description/lidar.xacro (robot description, xacro)
@@ -4,5 +4,5 @@
     <parent link="chassis"/>
     <child link="laser_frame"/>
-    <origin xyz="0.1 0 0.07" rpy="0 0 0"/>
+    <origin xyz="0.135 0 0.0915" rpy="0 0 0"/>
   </joint>
   <link name="laser_frame">

File: description/robot.urdf.xacro (robot description, xacro)
@@ -1,7 +1,12 @@
 <?xml version="1.0"?>
 <robot xmlns:xacro="http://www.ros.org/wiki/xacro"  name="robot">
+    <xacro:arg name="use_ros2_control" default="true"/>
     <xacro:include filename="robot_core.xacro" />
-    <!-- <xacro:include filename="gazebo_control.xacro"/> -->
-    <xacro:include filename="ros2_control.xacro"/>
+    <xacro:if value="$(arg use_ros2_control)">
+        <xacro:include filename="ros2_control.xacro"/>
+    </xacro:if>
+    <xacro:unless value="$(arg use_ros2_control)">
+        <xacro:include filename="gazebo_control.xacro"/>
+    </xacro:unless>
     <xacro:include filename="lidar.xacro"/>
 </robot>

File: description/robot_core.xacro (robot description, xacro)
@@ -63,5 +63,5 @@
     <collision>
       <geometry>
-        <cylinder radius="0.04" length="0.009" />
+        <sphere radius="0.04"/>
       </geometry>
     </collision>
@@ -89,5 +89,5 @@
     <collision>
       <geometry>
-        <cylinder radius="0.04" length="0.009" />
+        <sphere radius="0.04" />
       </geometry>
     </collision>

Commit message: Robot design change

File: description/lidar.xacro (robot description, xacro)
@@ -4,5 +4,5 @@
     <parent link="chassis"/>
     <child link="laser_frame"/>
-    <origin xyz="0.135 0 0.0915" rpy="0 0 0"/>
+    <origin xyz="0.0 0 0.0915" rpy="0 0 0"/>
   </joint>
   <link name="laser_frame">

File: description/robot_core.xacro (robot description, xacro)
@@ -35,18 +35,18 @@
   <link name="chassis">
     <visual>
-      <origin xyz="0.09 0 0.03" />
+      <origin xyz="0 0 0" />
       <geometry>
-        <box size="0.18 0.13 0.06" />
+        <box size="0.2 0.2 0.05" />
       </geometry>
       <material name="white" />
     </visual>
     <collision>
-      <origin xyz="0.09 0 0.03" />
+      <origin xyz="0 0 0" />
       <geometry>
-        <box size="0.18 0.13 0.06" />
+        <box size="0.2 0.2 0.05" />
       </geometry>
     </collision>
-    <xacro:inertial_box mass="0.5" x="0.18" y="0.13" z="0.06">
-      <origin xyz="0.09 0 0.3" rpy="0 0 0"/>
+    <xacro:inertial_box mass="0.5" x="0.2" y="0.2" z="0.05">
+      <origin xyz="0 0 0" rpy="0 0 0"/>
     </xacro:inertial_box>
   </link>
@@ -64,5 +64,5 @@
     <visual>
       <geometry>
-        <cylinder radius="0.04" length="0.009" />
+        <cylinder radius="0.0725" length="0.009" />
       </geometry>
       <material name="blue" />
@@ -70,8 +70,8 @@
     <collision>
       <geometry>
-        <sphere radius="0.04"/>
+        <sphere radius="0.0725"/>
       </geometry>
     </collision>
-    <xacro:inertial_cylinder mass="0.1" length="0.009" radius="0.04">
+    <xacro:inertial_cylinder mass="0.1" length="0.009" radius="0.0725">
       <origin xyz="0 0 0" rpy="0 0 0"/>
     </xacro:inertial_cylinder>
@@ -90,5 +90,5 @@
     <visual>
       <geometry>
-        <cylinder radius="0.04" length="0.009" />
+        <cylinder radius="0.0725" length="0.009" />
       </geometry>
       <material name="blue" />
@@ -96,8 +96,8 @@
     <collision>
       <geometry>
-        <sphere radius="0.04" />
+        <sphere radius="0.0725" />
       </geometry>
     </collision>
-    <xacro:inertial_cylinder mass="0.1" length="0.009" radius="0.04">
+    <xacro:inertial_cylinder mass="0.1" length="0.009" radius="0.0725">
       <origin xyz="0 0 0" rpy="0 0 0"/>
     </xacro:inertial_cylinder>
